Commit message: calibration seems working

File: fetch_description/robots/freight.urdf (robot description, URDF)
Before this commit: robot freight, 5 links, 4 joints
Links:
- added link base_camera_link
- added link base_camera_optical_frame
Joints:
- added joint base_camera_joint: type fixed, parent base_link, child base_camera_link, origin xyz=0.25 0 0.18 rpy= -0.19 3.141592653589793 -1.5707963267948966
- added joint base_camera_optical_joint: type fixed, parent base_camera_link, child base_camera_optical_frame, origin xyz=0 0 0 rpy=-1.5707963267966 0 0

Commit message: everything working

File: fetch_description/robots/freight.urdf (robot description, URDF)
Before this commit: robot freight, 7 links, 6 joints
Joints:
- joint base_camera_joint: origin xyz=0.25 0 0.18 rpy= -0.19 3.141592653589793 -1.5707963267948966 -> xyz=0.25 0 0.18 rpy= -0.19 3.4141592653589793 -1.5707963267948966

Commit message: clean up

File: fetch_description/robots/freight.urdf (robot description, URDF)
Before this commit: robot freight, 7 links, 6 joints
Links:
- removed link base_camera_link
- removed link base_camera_optical_frame
Joints:
- removed joint base_camera_joint
- removed joint base_camera_optical_joint
